Commit message: Update TESTPROJECT.xacro

File: TESTPROJECT/TESTPROJECT_description/urdf/TESTPROJECT.xacro (robot description, xacro)
@@ -94,5 +94,5 @@
   <parent link="base_link"/>
   <child link="left_wheel_1"/>
-  <axis xyz="0.0 0.0 -1.0"/>
+  <axis xyz="0.0 0.0 1.0"/>
 </joint>
 <joint name="Rigid3" type="fixed">
